File: eeprom.sch (KiCad schematic (older format))
At the start: 36 parts, among them SW1 SW_SPST, SW2 SW_DIP_x08, SW3 SW_DIP_x10, SW4 SW_DIP_x01, U3 74HC245, U4 M54513FP, U5 28C16

Commit message: Rename +5v global flags as 5V_SHARED
- moved 1x dip switch from place A0 to A10
Connections:
- net +5V is gone; now on net 5V_SHARED: C4.1, R2.2, R3.2, S1.3, U3.1 (A->B)
- net at D11.2 (A), R4.2, U5.8 (A0): now also SW3.1; no longer SW4.1
- net at D20.2 (A), RN3.10 (R9), U5.22 (A9): now also SW3.10; no longer SW3.2
- net at D21.2 (A), RN3.11 (R10), U5.19 (A10): now also SW4.1; no longer SW3.1
- net at D12.2 (A), RN3.2 (R1), U5.7 (A1): now also SW3.2; no longer SW3.10
- net at D13.2 (A), RN3.3 (R2), U5.6 (A2): now also SW3.3; no longer SW3.9
- net at D14.2 (A), RN3.4 (R3), U5.5 (A3): now also SW3.4; no longer SW3.8
- net at D15.2 (A), RN3.5 (R4), U5.4 (A4): now also SW3.5; no longer SW3.7
- net at D17.2 (A), RN3.7 (R6), U5.2 (A6): now also SW3.7; no longer SW3.5
- net at D18.2 (A), RN3.8 (R7), U5.1 (A7): now also SW3.8; no longer SW3.4
- net at D19.2 (A), RN3.9 (R8), U5.23 (A8): now also SW3.9; no longer SW3.3
Other:
- moved on the sheet: SW3, SW4
